File: gameboy-copperpilot.kicad_pcb (KiCad board)
At the start: 0 parts

Commit message: feat(hardware): complete 4-layer GKD Pixel ESP32-S3 console PCBA and enclosure
Implement complete hardware design, verified Lion Circuits 4-layer PCB layout (0 DRC errors, 100% routed), 6-block schematic capture (0 ERC errors), automated 35-point PyTest verification suite, turnkey PCBA manufacturing release generator, and parametric 3D snap-fit enclosure CAD models.

Co-Authored-By: CopperPilot <noreply@copperpilot.ai>
Parts:
- added C1: 10uF, C_0805_2012Metric, B.Cu at (31.5, 64.0)
- added C10: 100nF, C_0603_1608Metric, B.Cu at (31.5, 40.0)
- added C11: 22uF, C_0805_2012Metric, B.Cu at (45.5, 11.0)
- added C12: 100nF, C_0603_1608Metric, B.Cu at (49.0, 11.0)
- added C13: 1uF, C_0603_1608Metric, B.Cu at (45.5, 14.0)
- added C14: 10uF, C_0805_2012Metric, B.Cu at (48.0, 60.5)
- added C15: 100nF, C_0603_1608Metric, B.Cu at (51.5, 60.5)
- added C2: 100nF, C_0603_1608Metric, B.Cu at (31.5, 61.5)
- added C3: 4.7uF, C_0603_1608Metric, B.Cu at (20.0, 61.5)
- added C4: 10uF, C_0805_2012Metric, B.Cu at (48.0, 68.0)
- added C5: 100nF, C_0603_1608Metric, B.Cu at (51.0, 68.0)
- added C6: 100nF, C_0603_1608Metric, B.Cu at (15.0, 17.0)
- added C7: 10uF, C_0805_2012Metric, B.Cu at (43.0, 64.0)
- added C8: 100nF, C_0603_1608Metric, B.Cu at (43.0, 61.5)
- added C9: 22uF, C_0805_2012Metric, B.Cu at (27.0, 40.0)
- added D1: LED_RED, LED_0603_1608Metric, F.Cu at (29.5, 55.3)
- added D2: MBR0520, D_SOD-123, B.Cu at (25.0, 57.5)
- added D3: LED_GREEN, LED_0603_1608Metric, F.Cu at (33.5, 55.3)
- added J1: USB_C_Receptacle_USB2.0_16P, USB_C_Receptacle_GCT_USB4105-xx-A_16P_TopMnt_Horizontal, B.Cu at (31.5, 76.5)
- added J2: Conn_01x02, JST_PH_S2B-PH-K_1x02_P2.00mm_Horizontal, B.Cu at (15.0, 39.0)
- added J3: ILI9341_TFT_2.4in, ILI9341_TFT_2.4in_10P, F.Cu at (31.5, 46.0)
- added Q1: AO3401A, SOT-23, B.Cu at (20.0, 57.5)
- added Q2: 2N7002, SOT-23, B.Cu at (31.5, 36.0)
- added R1: 22, R_0603_1608Metric, B.Cu at (45.0, 25.5)
- added R10: 1k, R_0603_1608Metric, B.Cu at (48.0, 64.0)
- added R11: 10k, R_0603_1608Metric, B.Cu at (49.0, 14.0)
- added R12: 10k, R_0603_1608Metric, B.Cu at (17.5, 24.5)
- added R13: 10k, R_0603_1608Metric, B.Cu at (35.5, 42.0)
- added R14: 10, R_0805_2012Metric, B.Cu at (27.0, 36.0)
- added R15: 1k, R_0603_1608Metric, B.Cu at (35.5, 36.0)
- added R16: 100k, R_0603_1608Metric, B.Cu at (35.5, 39.0)
- added R17: 10k, R_0603_1608Metric, B.Cu at (8.00, 49.0)
- added R18: 10k, R_0603_1608Metric, B.Cu at (10.5, 49.0)
- added R19: 10k, R_0603_1608Metric, B.Cu at (13.0, 49.0)
- added R2: 22, R_0603_1608Metric, B.Cu at (45.0, 28.0)
- added R20: 10k, R_0603_1608Metric, B.Cu at (15.5, 49.0)
- added R21: 10k, R_0603_1608Metric, B.Cu at (18.0, 49.0)
- added R22: 10k, R_0603_1608Metric, B.Cu at (52.0, 49.0)
- added R23: 10k, R_0603_1608Metric, B.Cu at (42.0, 49.0)
- added R24: 10k, R_0603_1608Metric, B.Cu at (44.5, 49.0)
- added R25: 10k, R_0603_1608Metric, B.Cu at (47.0, 49.0)
- added R26: 10k, R_0603_1608Metric, B.Cu at (49.5, 49.0)
- added R27: 10k, R_0603_1608Metric, B.Cu at (20.5, 49.0)
- added R28: 10k, R_0603_1608Metric, B.Cu at (23.0, 49.0)
- added R29: 10k, R_0603_1608Metric, B.Cu at (54.5, 49.0)
- added R3: 5.1k, R_0603_1608Metric, B.Cu at (25.0, 71.5)
- added R30: 10k, R_0603_1608Metric, B.Cu at (57.0, 49.0)
- added R4: 5.1k, R_0603_1608Metric, B.Cu at (38.0, 71.5)
- added R5: 1k, R_0603_1608Metric, B.Cu at (20.0, 64.0)
- added R6: 2.0k 1%, R_0603_1608Metric, B.Cu at (15.0, 68.0)
- added R7: 100k, R_0603_1608Metric, B.Cu at (15.0, 57.5)
- added R8: 100k 1%, R_0603_1608Metric, B.Cu at (15.0, 12.0)
- added R9: 100k 1%, R_0603_1608Metric, B.Cu at (15.0, 14.5)
- added SW1: SW_SPDT, SW_SPDT_PCM12, B.Cu at (59.5, 23.2)
- added SW10: A, SW_SPST_PTS645Sx43SMTR92, F.Cu at (54.5, 61.8)
- added SW11: B, SW_SPST_PTS645Sx43SMTR92, F.Cu at (47.9, 68.0)
- added SW12: SELECT, SW_Tactile_SPST_NO_Straight_CK_PTS636Sx25SMTRLFS, F.Cu at (27.2, 67.4)
- added SW13: START, SW_Tactile_SPST_NO_Straight_CK_PTS636Sx25SMTRLFS, F.Cu at (35.3, 66.5)
- added SW14: L1, SW_SPST_B3U-3000P, F.Cu at (9.50, 2.20)
- added SW15: L2, SW_SPST_B3U-3000P, F.Cu at (18.3, 2.20)
- added SW16: R2, SW_SPST_B3U-3000P, F.Cu at (44.7, 2.20)
- added SW17: R1, SW_SPST_B3U-3000P, F.Cu at (53.5, 2.20)
- added SW2: RESET, SW_Tactile_SPST_NO_Straight_CK_PTS636Sx25SMTRLFS, B.Cu at (54.5, 13.5)
- added SW3: BOOT, SW_Tactile_SPST_NO_Straight_CK_PTS636Sx25SMTRLFS, B.Cu at (12.5, 27.5)
- added SW4: UP, SW_SPST_PTS645Sx43SMTR92, F.Cu at (14.7, 54.7)
- added SW5: DOWN, SW_SPST_PTS645Sx43SMTR92, F.Cu at (14.7, 67.3)
- added SW6: LEFT, SW_SPST_PTS645Sx43SMTR92, F.Cu at (8.35, 61.0)
- added SW7: RIGHT, SW_SPST_PTS645Sx43SMTR92, F.Cu at (20.9, 61.0)
- added SW8: X, SW_SPST_PTS645Sx43SMTR92, F.Cu at (48.0, 55.4)
- added SW9: Y, SW_SPST_PTS645Sx43SMTR92, F.Cu at (41.4, 61.7)
- added U1: USBLC6-2SC6, SOT-23-6, B.Cu at (31.5, 68.0)
- added U2: MCP73831-2-OT, SOT-23-5, B.Cu at (20.0, 68.0)
- added U3: AP2112K-3.3, SOT-23-5, B.Cu at (43.0, 68.0)
- added U4: ESP32-S3-WROOM-1, ESP32-S3-WROOM-1, B.Cu at (31.5, 16.0)
Routing:
- net GND: track 0.00 -> 509.4 mm, vias 0 -> 2
- net /+3V3: track 0.00 -> 172.7 mm, vias 0 -> 4
- net /BTN_DOWN: track 0.00 -> 103.8 mm, vias 0 -> 3
- net /VSYS: track 0.00 -> 99.2 mm, vias 0 -> 3
- net /BTN_L1: track 0.00 -> 90.9 mm, vias 0 -> 3
- net /VSYS_PRE: track 0.00 -> 87.0 mm, vias 0 -> 3
- net /BTN_Y: track 0.00 -> 83.8 mm, vias 0 -> 2
- net /BTN_R1: track 0.00 -> 82.8 mm, vias 0 -> 3
- net /BTN_LEFT: track 0.00 -> 80.5 mm, vias 0 -> 2
- net /BTN_B: track 0.00 -> 80.1 mm, vias 0 -> 2
- net /BTN_RIGHT: track 0.00 -> 75.1 mm, vias 0 -> 3
- net /BTN_A: track 0.00 -> 74.5 mm, vias 0 -> 3
- net /BTN_R2: track 0.00 -> 70.8 mm, vias 0 -> 2
- net /BTN_X: track 0.00 -> 70.6 mm, vias 0 -> 3
- net /BTN_UP: track 0.00 -> 70.2 mm, vias 0 -> 2
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- added copper zone on B.Cu, net GND
- added copper zone on F.Cu, net GND
- added copper zone on In1.Cu, net GND
Other:
- board outline added: 63 x 80 mm
- copper layers 0 -> 4
