File: gameboy-copperpilot.kicad_sch (KiCad schematic)
At the start: 0 parts

Commit message: feat(hardware): complete 4-layer GKD Pixel ESP32-S3 console PCBA and enclosure
Implement complete hardware design, verified Lion Circuits 4-layer PCB layout (0 DRC errors, 100% routed), 6-block schematic capture (0 ERC errors), automated 35-point PyTest verification suite, turnkey PCBA manufacturing release generator, and parametric 3D snap-fit enclosure CAD models.

Co-Authored-By: CopperPilot <noreply@copperpilot.ai>
Parts:
- added C1, C14, C4, C7: 10uF, Capacitor_SMD:C_0805_2012Metric, symbol Device:C
- added C10, C12, C15, C2, C5, C6, C8: 100nF, Capacitor_SMD:C_0603_1608Metric, symbol Device:C
- added C11, C9: 22uF, Capacitor_SMD:C_0805_2012Metric, symbol Device:C
- added C13: 1uF, Capacitor_SMD:C_0603_1608Metric, symbol Device:C
- added C3: 4.7uF, Capacitor_SMD:C_0603_1608Metric, symbol Device:C
- added D1: LED_RED, LED_SMD:LED_0603_1608Metric, symbol Device:LED
- added D2: MBR0520, Diode_SMD:D_SOD-123, symbol Diode:SS14
- added D3: LED_GREEN, LED_SMD:LED_0603_1608Metric, symbol Device:LED
- added J1: USB_C_Receptacle_USB2.0_16P, Connector_USB:USB_C_Receptacle_GCT_USB4105-xx-A_16P_TopMnt_Horizontal, symbol Connector:USB_C_Receptacle_USB2.0_16P
- added J2: Conn_01x02, Connector_JST:JST_PH_S2B-PH-K_1x02_P2.00mm_Horizontal, symbol Connector_Generic:Conn_01x02
- added J3: ILI9341_TFT_2.4in, gameboy_handheld:ILI9341_TFT_2.4in_10P, symbol gameboy_handheld:ILI9341_TFT_2.4in
- added Q1: AO3401A, Package_TO_SOT_SMD:SOT-23, symbol Transistor_FET:Q_PMOS_GSD
- added Q2: 2N7002, Package_TO_SOT_SMD:SOT-23, symbol Transistor_FET:Q_NMOS_GSD
- added R1, R2: 22, Resistor_SMD:R_0603_1608Metric, symbol Device:R
- added R10, R15, R5: 1k, Resistor_SMD:R_0603_1608Metric, symbol Device:R
- added R11, R12, R13, R17, R18, R19, R20, R21, R22, R23, R24, R25, R26, R27, R28, R29, R30: 10k, Resistor_SMD:R_0603_1608Metric, symbol Device:R
- added R14: 10, Resistor_SMD:R_0805_2012Metric, symbol Device:R
- added R16, R7: 100k, Resistor_SMD:R_0603_1608Metric, symbol Device:R
- added R3, R4: 5.1k, Resistor_SMD:R_0603_1608Metric, symbol Device:R
- added R6: 2.0k 1%, Resistor_SMD:R_0603_1608Metric, symbol Device:R
- added R8, R9: 100k 1%, Resistor_SMD:R_0603_1608Metric, symbol Device:R
- added SW1: SW_SPDT, Button_Switch_SMD:SW_SPDT_PCM12, symbol Switch:SW_SPDT
- added SW10: A, Button_Switch_SMD:SW_SPST_PTS645Sx43SMTR92, symbol Switch:SW_Push
- added SW11: B, Button_Switch_SMD:SW_SPST_PTS645Sx43SMTR92, symbol Switch:SW_Push
- added SW12: SELECT, Button_Switch_SMD:SW_Tactile_SPST_NO_Straight_CK_PTS636Sx25SMTRLFS, symbol Switch:SW_Push
- added SW13: START, Button_Switch_SMD:SW_Tactile_SPST_NO_Straight_CK_PTS636Sx25SMTRLFS, symbol Switch:SW_Push
- added SW14: L1, Button_Switch_SMD:SW_SPST_B3U-3000P, symbol Switch:SW_Push
- added SW15: L2, Button_Switch_SMD:SW_SPST_B3U-3000P, symbol Switch:SW_Push
- added SW16: R2, Button_Switch_SMD:SW_SPST_B3U-3000P, symbol Switch:SW_Push
- added SW17: R1, Button_Switch_SMD:SW_SPST_B3U-3000P, symbol Switch:SW_Push
- added SW2: RESET, Button_Switch_SMD:SW_Tactile_SPST_NO_Straight_CK_PTS636Sx25SMTRLFS, symbol Switch:SW_Push
- added SW3: BOOT, Button_Switch_SMD:SW_Tactile_SPST_NO_Straight_CK_PTS636Sx25SMTRLFS, symbol Switch:SW_Push
- added SW4: UP, Button_Switch_SMD:SW_SPST_PTS645Sx43SMTR92, symbol Switch:SW_Push
- added SW5: DOWN, Button_Switch_SMD:SW_SPST_PTS645Sx43SMTR92, symbol Switch:SW_Push
- added SW6: LEFT, Button_Switch_SMD:SW_SPST_PTS645Sx43SMTR92, symbol Switch:SW_Push
- added SW7: RIGHT, Button_Switch_SMD:SW_SPST_PTS645Sx43SMTR92, symbol Switch:SW_Push
- added SW8: X, Button_Switch_SMD:SW_SPST_PTS645Sx43SMTR92, symbol Switch:SW_Push
- added SW9: Y, Button_Switch_SMD:SW_SPST_PTS645Sx43SMTR92, symbol Switch:SW_Push
- added U1: USBLC6-2SC6, Package_TO_SOT_SMD:SOT-23-6, symbol Power_Protection:USBLC6-2SC6
- added U2: MCP73831-2-OT, Package_TO_SOT_SMD:SOT-23-5, symbol Battery_Management:MCP73831-2-OT
- added U3: AP2112K-3.3, Package_TO_SOT_SMD:SOT-23-5, symbol Regulator_Linear:AP2112K-3.3
- added U4: ESP32-S3-WROOM-1, RF_Module:ESP32-S3-WROOM-1, symbol RF_Module:ESP32-S3-WROOM-1
Connections:
- new net: Q2.1 (G), R15.2, R16.1
- new net: Q2.3 (D), R14.2
- new net: R6.2, U2.5 (PROG)
- new net: J1.B5 (CC2), R4.1
- new net: R2.1, U1.6 (I/O1)
- new net: R1.1, U1.4 (I/O2)
- new net: J3.10 (LED_K), R14.1
- new net: J1.A5 (CC1), R3.1
- new net: J1.A6 (D+), J1.B6 (D+), U1.3 (I/O2)
- new net: J1.A7 (D-), J1.B7 (D-), U1.1 (I/O1)
- new net +3V3: C10.1, C11.1, C12.1, C14.1, C15.1, C9.1, J3.1 (VCC), J3.9 (LED_A), R10.1, R11.1, R12.2, R13.1, R17.1, R18.1, R19.1, R20.1, R21.1, R22.1, R23.1, R24.1, R25.1, R26.1, R27.1, R28.1, R29.1, R30.1, U3.5 (VOUT), U4.2 (3V3)
- new net BOOT_BTN: R12.1, SW3.2, U4.27 (IO0)
- new net BTN_A: R23.2, SW10.1, U4.34 (IO41)
- new net BTN_B: R24.2, SW11.1, U4.35 (IO42)
- new net BTN_DOWN: R18.2, SW5.1, U4.5 (IO5)
- new net BTN_L1: R27.2, SW14.1, U4.8 (IO15)
- new net BTN_L2: R28.2, SW15.1, U4.24 (IO47)
- new net BTN_LEFT: R19.2, SW6.1, U4.6 (IO6)
- new net BTN_R1: R30.2, SW17.1, U4.31 (IO38)
- new net BTN_R2: R29.2, SW16.1, U4.25 (IO48)
- new net BTN_RIGHT: R20.2, SW7.1, U4.7 (IO7)
- new net BTN_SELECT: R25.2, SW12.1, U4.9 (IO16)
- new net BTN_START: R26.2, SW13.1, U4.10 (IO17)
- new net BTN_UP: R17.2, SW4.1, U4.4 (IO4)
- new net BTN_X: R21.2, SW8.1, U4.32 (IO39)
- new net BTN_Y: R22.2, SW9.1, U4.33 (IO40)
- new net CHG_STAT: D1.1 (K), D1.2 (A), R5.1, U2.1 (STAT), U4.38 (IO2)
- new net CHIP_EN: C13.1, R11.2, SW2.2, U4.3 (EN)
- new net GND: C1.2, C10.2, C11.2, C12.2, C13.2, C14.2, C15.2, C2.2, C3.2, C4.2, C5.2, C6.2, C7.2, C8.2, C9.2, D3.1 (K), D3.2 (A), J1.A1 (GND), J1.A12 (GND), J1.B1 (GND), J1.B12 (GND), J1.S1 (SHIELD), J2.2 (Pin_2), J3.2 (GND), Q2.2 (S), R10.2, R16.2, R3.2, R4.2, R6.1, R7.2, R9.2, SW10.2, SW11.2, SW12.2, SW13.2, SW14.2, SW15.2, SW16.2, SW17.2, SW2.1, SW3.1, SW4.2, SW5.2, SW6.2, SW7.2, SW8.2, SW9.2, U1.2 (GND), U2.2 (V_{SS}), U3.2 (GND), U4.1 (GND), U4.40 (GND), U4.41 (GND)
- new net TFT_BL: R15.1, U4.23 (IO21)
- new net TFT_CS: J3.3 (CS), R13.2, U4.18 (IO10)
- new net TFT_DC: J3.5 (DC), U4.17 (IO9)
- new net TFT_MISO: J3.8 (MISO), U4.21 (IO13)
- new net TFT_MOSI: J3.6 (MOSI), U4.19 (IO11)
- new net TFT_RST: J3.4 (RESET), U4.22 (IO14)
- new net TFT_SCLK: J3.7 (SCLK), U4.20 (IO12)
- new net USB_D+: R1.2, U4.14 (USB_D+)
- new net USB_D-: R2.2, U4.13 (USB_D-)
- new net VBAT: C3.1, J2.1 (Pin_1), Q1.3 (D), U2.3 (V_{BAT})
- new net VBAT_SENSE: C6.1, R8.2, R9.1, U4.39 (IO1)
- new net VBUS: C1.1, C2.1, C4.1, C5.1, D2.1 (K), D2.2 (A), J1.A4 (VBUS), J1.A9 (VBUS), J1.B4 (VBUS), J1.B9 (VBUS), Q1.1 (G), Q1.2 (S), R5.2, R7.1, SW1.2 (B), U1.5 (VBUS), U2.4 (V_{DD})
- new net VSYS: C7.1, C8.1, R8.1, SW1.3 (C), U3.1 (VIN), U3.3 (EN)
- no-connect marks 0 -> 14
Other:
- note added: "CONTROLS: 14 Active-Low Gameplay & Shoulder Switches"
- note added: "DISPLAY: 2.4-inch 320x240 ILI9341 SPI TFT & Backlight"
- note added: "MCU: ESP32-S3-WROOM-1 Host & Boot Strapping"
- note added: "POWER: Automatic Load-Sharing & AP2112K-3.3 LDO"
- note added: "POWER: USB-C 5V Input, ESD Protection & LiPo Charger"
