File: copperpilot-retro-handheld.kicad_sch (KiCad schematic)
At the start: 74 parts, among them J1 USB_C_Receptacle_USB2.0_16P, J2 Conn_01x02, J3 ILI9341_TFT_2.4in, Q1 AO3401A, Q2 2N7002, SW1 SW_SPDT, SW10 A, SW11 B, SW12 SELECT, SW13 START, SW14 L1, SW15 L2, SW16 R2, SW17 R1, SW2 RESET, SW3 BOOT, SW4 UP, SW5 DOWN, SW6 LEFT, SW7 RIGHT, SW8 X, SW9 Y, U1 USBLC6-2SC6, U2 MCP73831-2-OT, U3 AP2112K-3.3, U4 ESP32-S3-WROOM-1

Commit message: chore: rename project from gameboy-copperpilot to copperpilot-retro-handheld
Remove trademarked "gameboy" naming from the repo: KiCad project files,
custom symbol/footprint library, PCBA 3D models (incl. embedded STEP/GLB
names), build scripts, tests, README and LICENSE.

Co-Authored-By: CopperPilot <noreply@copperpilot.ai>
Parts:
- J3: footprint gameboy_handheld:ILI9341_TFT_2.4in_10P -> copperpilot_retro_handheld:ILI9341_TFT_2.4in_10P; symbol gameboy_handheld:ILI9341_TFT_2.4in -> copperpilot_retro_handheld:ILI9341_TFT_2.4in
Changed lines of the file:
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@@
 	)
 	(symbol
-		(lib_id "gameboy_handheld:ILI9341_TFT_2.4in")
+		(lib_id "copperpilot_retro_handheld:ILI9341_TFT_2.4in")
 		(at 335.28 63.5 0)
 		(unit 1)
@@
 		)
 		(property "Footprint"
-			"gameboy_handheld:ILI9341_TFT_2.4in_10P"
+			"copperpilot_retro_handheld:ILI9341_TFT_2.4in_10P"
 			(at 335.28 63.5 0)
 			(hide yes)
